Commit message: creature

File: body.urdf (robot description, URDF)
Before this commit: robot robot, 9 links, 8 joints
Links:
- removed link BackLeg
- removed link FrontLeg
- removed link LeftLeg
- removed link LowerBackLeg
- removed link LowerFrontLeg
- removed link LowerLeftLeg
- removed link LowerRightLeg
- added link Platform, mass 0.1; collision box size=1 1 0.1; visual box size=1 1 0.1
- added link RightLeg2, mass 0.1; collision box size=0.2 0.5 0.2; visual box size=0.2 0.5 0.2
- added link RightLeg3, mass 0.1; collision box size=0.2 0.5 0.2; visual box size=0.2 0.5 0.2
- added link RightLeg4, mass 0.1; collision box size=0.2 0.5 0.2; visual box size=0.2 0.5 0.2
- added link RightLeg5, mass 0.1; collision box size=0.2 0.5 0.2; visual box size=0.2 0.5 0.2
- link RightLeg: mass 1 -> 0.1; geometry collision box size=0.2 0.5 0.2; visual box size=0.2 0.5 0.2
- link Torso: mass 1 -> 999; geometry collision box size=2 1 1; visual box size=2 1 1
Joints:
- removed joint BackLeg_LowerBackLeg
- removed joint FrontLeg_LowerFrontLeg
- removed joint LeftLeg_LowerLeftLeg
- removed joint RightLeg_LowerRightLeg
- removed joint Torso_BackLeg
- removed joint Torso_FrontLeg
- removed joint Torso_LeftLeg
- added joint RightLeg2_RightLeg3: type revolute, parent RightLeg2, child RightLeg3, origin xyz=0 0.5 0 rpy=0 0 0, axis 1 0 0, limit lower=-3.14159 upper=3.14159 effort=0.0 velocity=0.0
- added joint RightLeg3_RightLeg4: type revolute, parent RightLeg3, child RightLeg4, origin xyz=0 0.5 0 rpy=0 0 0, axis 1 0 0, limit lower=-3.14159 upper=3.14159 effort=0.0 velocity=0.0
- added joint RightLeg4_RightLeg5: type revolute, parent RightLeg4, child RightLeg5, origin xyz=0 0.5 0 rpy=0 0 0, axis 1 0 0, limit lower=-3.14159 upper=3.14159 effort=0.0 velocity=0.0
- added joint RightLeg5_Platform: type revolute, parent RightLeg5, child Platform, origin xyz=0 0.5 0 rpy=0 0 0, axis 1 0 0, limit lower=-3.14159 upper=3.14159 effort=0.0 velocity=0.0
- added joint RightLeg_RightLeg2: type revolute, parent RightLeg, child RightLeg2, origin xyz=0 0.5 0 rpy=0 0 0, axis 1 0 0, limit lower=-3.14159 upper=3.14159 effort=0.0 velocity=0.0
- joint Torso_RightLeg: axis 0 1 0 -> 1 0 0; origin xyz=0.5 0 1 rpy=0 0 0 -> xyz=0.0 0.5 1 rpy=0 0 0
